File: ee599_4/ee599_4.kicad_pcb (KiCad board)
At the start: 4 copper layers, 47.5 x 39.9 mm, 5 parts, among them J0 TS-105-G-A, J1 60312202114512, J2 60312202114512

Commit message: started minjings, still need to work on it
Parts:
- added C2: 10uF, Capacitor_SMD:C_0603_1608Metric, F.Cu at (94.0, 92.8)
- added C3: 100pF, Capacitor_SMD:C_0603_1608Metric, F.Cu at (96.2, 92.8)
- added C4: 100pF, Capacitor_SMD:C_0603_1608Metric, F.Cu at (111.2, 98.6)
- added C5: 10uF, Capacitor_SMD:C_0603_1608Metric, F.Cu at (168.4, 95.4)
- added C6: 100pF, Capacitor_SMD:C_0603_1608Metric, F.Cu at (168.4, 97.9)
- added J3: Conn_01x02_Pin, Connector_PinHeader_2.54mm:PinHeader_1x02_P2.54mm_Vertical, F.Cu at (83.6, 91.9)
- added J4: 60312202114512, foot:60312202114512, F.Cu at (95.0, 76.9)
- added J5: 60312202114512, foot:60312202114512, F.Cu at (108.3, 76.9)
- C1: value 1uF -> 10uF
- moved C1 2.22 mm to (113.2, 98.6)
Connections:
- EE1 pad 56: GND -> fVCO_180_Min
- EE1 pad 57: GND -> unconnected-(EE1-FVCO_Min-Pad57)
- EE1 pad 58: GND -> fVCO_0_Min
- EE1 pad 59: GND -> unconnected-(EE1-OUTN_Min-Pad59)
- EE1 pad 60: GND -> unconnected-(EE1-OUTP_Min-Pad60)
- EE1 pad 61: GND -> VDD_Min
Routing:
- net VDD_Min: track 0.00 -> 14.7 mm
- net fVCO_180_Min: track 0.00 -> 14.5 mm
- net fVCO_0_Min: track 0.00 -> 13.6 mm
- net GND: track 21.6 -> 26.1 mm, vias 210 -> 175

Commit message: minjing osc layout
Parts:
- added C7: 10uF, Capacitor_SMD:C_0603_1608Metric, F.Cu at (101.4, 85.0)
- added C8: 100pF, Capacitor_SMD:C_0603_1608Metric, F.Cu at (101.4, 86.8)
- C5, C6: moved to B.Cu
- J3: value Conn_01x02_Pin -> Conn_01x03_Pin; footprint Connector_PinHeader_2.54mm:PinHeader_1x02_P2.54mm_Vertical -> Connector_PinHeader_2.54mm:PinHeader_1x03_P2.54mm_Vertical
- moved C6 60.3 mm to (108.3, 102.7), turned to 90 degrees
- moved C5 58.5 mm to (110.3, 102.7), turned to 90 degrees
- moved J3 0.52 mm to (84.0, 91.5)
Connections:
- EE1 pad 57: unconnected-(EE1-FVCO_Min-Pad57) -> VC_Min
- EE1 pad 77: GND -> (no net)
- EE1 pad 78: GND -> (no net)
- EE1 pad 79: GND -> (no net)
- EE1 pad 80: GND -> (no net)
- EE1 pad 81: GND -> (no net)
Routing:
- net VC_Min: track 0.00 -> 25.0 mm, vias 0 -> 1
- net GND: vias 175 -> 165
