File: ee599_4/ee599_4.kicad_sch (KiCad schematic)
At the start: 6 parts, among them J1 out_0, J2 out_180

Commit message: :0
Parts:
- removed C2, C3: 1uF, symbol Device:C
- removed J1: out_0, symbol Connector:Conn_Coaxial
- removed J2: out_180, symbol Connector:Conn_Coaxial
- added J0: TS-105-G-A, CON5_1X5_TU_HTS_SAI, symbol lib:TS-105-G-A
- added J1, J2: 60312202114512, foot:60312202114512, symbol lib:60312202114512
- C1: footprint (none) -> Capacitor_SMD:C_0603_1608Metric
Connections:
- net VDC is gone; now on net VDD_Mel: C1.1
- net F0_Mel: now also J2.1
- net GND: now also EE1.1 (Vdd_TIFet), EE1.16 (Amp_Out+), EE1.17 (AMP_IN-), EE1.18 (AMP_IN+), EE1.19 (AMP_Out-), EE1.2 (Out_TIFet), EE1.20 (VC_Hay), EE1.21 (NC), EE1.22 (NC), EE1.23 (NC), EE1.24 (VS_Hay), EE1.27 (A1_Hay), EE1.28 (A2_Hay), EE1.29 (A3_Hay), EE1.3 (VC_Kai), EE1.30 (AMP_CLK00), EE1.31 (T2_Jam), EE1.32 (T1_Jam), EE1.33 (VS_Jam), EE1.35 (VDD_Bar), EE1.36 (VC_Jam), EE1.37 (NC), EE1.38 (NC), EE1.39 (NC), EE1.4 (VS_Kai), EE1.40 (NC), EE1.41 (A1_Bar), EE1.42 (B2_Bar), EE1.43 (B0_Bar), EE1.44 (VS_Bar), EE1.45 (VC_Bar), EE1.46 (A0_Bar), EE1.47 (B1_Bar), EE1.48 (B1_Sim), EE1.49 (B2_Sim), EE1.5 (VC_Jae), EE1.50 (A2_Sim), EE1.51 (A1_Sim), EE1.52 (VS_Sim), EE1.53 (VS_Jae), EE1.54 (VDD_Jae), EE1.55 (Voutp2_Jae), EE1.56 (fVCO_180_Min), EE1.57 (FVCO_Min), EE1.58 (fVCO_0_Min), EE1.59 (OUTN_Min), EE1.60 (OUTP_Min), EE1.61 (VDD_Min), EE1.62 (NC), EE1.63 (NC), EE1.64 (VS_Hay), EE1.66 (Out_Hua), EE1.67 (VS_Hua), EE1.69 (TN2_Kai), EE1.7 (Voutp_Jae), EE1.70 (TN1_Kai), EE1.71 (TP3_Kai), EE1.72 (TP2_Kai), EE1.73 (TP1_Kai), EE1.74 (VDD_Kai/Hua), EE1.76 (Out_Hua), EE1.77 (VC_Hua), EE1.78 (NC), EE1.79 (NC), EE1.8 (VDD_Sim), EE1.80 (IN_TiFet), EE1.81 (GNDPLATE), EE1.9 (VC_Sim), J0.4, J1.2, J2.2
- net VC_Mel: now also J0.2
- net VS_Mel: now also J0.1
- net f180_Mel: now also J1.1
- net VDD_Mel: now reaches EE1.25 (VDD_Mel)
- net VDD_Mel: now also J0.3
- no-connect marks 67 -> 1
Other:
- moved on the sheet: C1

Commit message: started minjings, still need to work on it
Parts:
- added C2, C5: 10uF, Capacitor_SMD:C_0603_1608Metric, symbol Device:C
- added C3, C4, C6: 100pF, Capacitor_SMD:C_0603_1608Metric, symbol Device:C
- added J3: Conn_01x02_Pin, Connector_PinHeader_2.54mm:PinHeader_1x02_P2.54mm_Vertical, symbol Connector:Conn_01x02_Pin
- added J4, J5: 60312202114512, foot:60312202114512, symbol lib:60312202114512
- C1: value 1uF -> 10uF
Connections:
- net GND: now also C2.2, C3.2, C4.2, C5.2, C6.2, J3.2 (Pin_2), J4.2, J5.2; no longer EE1.56 (fVCO_180_Min), EE1.57 (FVCO_Min), EE1.58 (fVCO_0_Min), EE1.59 (OUTN_Min), EE1.60 (OUTP_Min), EE1.61 (VDD_Min)
- net VC_Mel: now also C5.1, C6.1
- net VDD_Mel: now also C4.1
- new net VDD_Min: C2.1, C3.1, EE1.61 (VDD_Min), J3.1 (Pin_1)
- new net fVCO_0_Min: EE1.58 (fVCO_0_Min), J4.1
- new net fVCO_180_Min: EE1.56 (fVCO_180_Min), J5.1
Other:
- moved on the sheet: C1, J0, J1, J2

Commit message: minjing osc layout
Parts:
- removed J3: Conn_01x02_Pin, Connector_PinHeader_2.54mm:PinHeader_1x02_P2.54mm_Vertical, symbol Connector:Conn_01x02_Pin
- added C7: 10uF, Capacitor_SMD:C_0603_1608Metric, symbol Device:C
- added C8: 100pF, Capacitor_SMD:C_0603_1608Metric, symbol Device:C
- added J3: Conn_01x03_Pin, Connector_PinHeader_2.54mm:PinHeader_1x03_P2.54mm_Vertical, symbol Connector:Conn_01x03_Pin
- J1, J2, J4, J5: footprint foot:60312202114512 -> 60312202114512:60312202114512
Connections:
- net GND: now also EE1. (GNDPLATE), C7.2, C8.2, J3.2 (Pin_2); no longer EE1.77 (VC_Hua), EE1.78 (NC), EE1.79 (NC), EE1.80 (IN_TiFet), EE1.81 (GNDPLATE)
- net VDD_Min: now also J3.1 (Pin_1)
- net VC_Min: now reaches EE1.57 (VC_Min)
- net VC_Min: now also C7.1, C8.1, J3.3 (Pin_3)
- no-connect marks 1 -> 3
Other:
- moved on the sheet: J4, J5
